File: Incubator-PowerBoard.kicad_pcb (KiCad board)
At the start: 2 copper layers, 96.5 x 61 mm, 29 parts, among them J1 Conn_01x12_Socket, J10 LIGHTS, J12 Conn_01x02_Pin, J13 ATX-24, J2 Conn_01x16_Socket, J3 OUT_FAN_1, J4 OUT_FAN_2, J5 IN_FAN_1, J6 IN_FAN_2, J7 Conn_01x08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

Commit message: changes
Parts:
- removed J7: Conn_01x08, Connector_PinHeader_2.54mm:PinHeader_1x08_P2.54mm_Vertical
- added J11: Conn_02x10_Odd_Even, Connector_PinHeader_2.54mm:PinHeader_2x10_P2.54mm_Vertical, F.Cu at (147.3, 30.5)
- added R10: 0R, Resistor_SMD:R_0603_1608Metric, F.Cu at (144.8, 62.6)
- added R11: 0R, Resistor_SMD:R_0603_1608Metric, F.Cu at (147.3, 62.6)
- added R6: 0R, Resistor_SMD:R_0603_1608Metric, F.Cu at (157.5, 62.5)
- added R7: 0R, Resistor_SMD:R_0603_1608Metric, F.Cu at (154.9, 62.5)
- added R8: 0R, Resistor_SMD:R_0603_1608Metric, F.Cu at (152.4, 62.5)
- added R9: 0R, Resistor_SMD:R_0603_1608Metric, F.Cu at (142.2, 62.5)
- moved J8 3.30 mm to (163.3, 64.8)
- moved J12 2.54 mm to (175.3, 30.5)
- moved R5 0.80 mm to (150.4, 62.5), turned to 90 degrees
Connections:
- J1 pad 4: unconnected-(J1-Pin_4-Pad4) -> /IO13
- J1 pad 5: unconnected-(J1-Pin_5-Pad5) -> /IO12
- J2 pad 11: /PWM_L -> /SCK
- J2 pad 12: /PWM_FAN_IN_1 -> /MOSI
- J2 pad 13: /PWM_FAN_IN_2 -> /MISO
- J2 pad 5: unconnected-(J2-Pin_5-Pad5) -> /AO
- J2 pad 6: unconnected-(J2-Pin_6-Pad6) -> /A1
- J2 pad 7: unconnected-(J2-Pin_7-Pad7) -> Net-(J2-Pin_7)
- J2 pad 8: unconnected-(J2-Pin_8-Pad8) -> Net-(J2-Pin_8)
- J2 pad 9: unconnected-(J2-Pin_9-Pad9) -> Net-(J2-Pin_9)
Routing:
- net /MISO: track 0.00 -> 119.0 mm
- net /MOSI: track 0.00 -> 110.4 mm
- net /SCK: track 0.00 -> 103.4 mm
- net /A1: track 0.00 -> 45.5 mm
- net /AO: track 0.00 -> 44.0 mm
- net /IO12: track 0.00 -> 17.8 mm
- net /IO13: track 0.00 -> 17.3 mm
- net /PWM_L: track 40.3 -> 56.8 mm
- net +5V: track 0.00 -> 10.9 mm, vias 0 -> 4
- net Net-(J2-Pin_9): track 0.00 -> 3.37 mm
- net Net-(J2-Pin_8): track 0.00 -> 3.37 mm
- net Net-(J2-Pin_7): track 0.00 -> 3.24 mm
- net /TACH_1: track 38.7 -> 36.6 mm
- net /TOGGLE_COOL_1: track 62.1 -> 64.0 mm
- net /PS_ON: track 20.2 -> 19.2 mm
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
Commit message: adding MFG files
Parts:
- removed the G*** at (160.0, 53.3)
- added G***: LOGO, openplantIncubator_fp:DNA_silk_fp_1, B.Cu at (160.3, 49.5)
Other:
- board text added: "3V3"
- board text added: "A0"
- board text added: "A1"
- board text added: "ALT"
- board text added: "B1"
- board text added: "B2"
- board text added: "B3"
- board text added: "D13"
- board text added: "MISO"
- board text added: "MOSI"
- board text added: "NC"
- board text added: "SCK"
- board text added: "SCL"
- board text added: "SDA"
