File: Incubator-PowerBoard.kicad_sch (KiCad schematic)
At the start: 14 parts, among them J1 Conn_01x12_Socket, J2 Conn_01x16_Socket, J3 Conn_01x04_Pin, J4 Conn_01x04_Pin, J5 Conn_01x04_Pin, J6 Conn_01x04_Pin, J7 Conn_01x08, Q1 2N7002E, Q2 2N7002E, Q3 2N7002E, Q4 2N7002E, Q5 2N7002E

Commit message: udpated comments
Other:
- note added: "ToDO: 1. Add 24 pin ATX connector 2. Add provision for beakout board for display and input controls - Needs 3v3 from ATX going to the display 3. find switches"
Changed lines of the file:
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@@
     (effects (font (size 0.75 0.75)) (justify left bottom))
+  )
+  (text "ToDO:\n1. Add 24 pin ATX connector\n2. Add provision for beakout board for display and input controls\n  - Needs 3v3 from ATX going to the display\n3. find switches"
+    (at 120.015 26.035 0)
+    (effects (font (size 1.27 1.27)) (justify left bottom))
   )
   (text "SET_LIGHT_DOWN" (at 50.8 83.185 0)

Commit message: layout complete
Parts:
- added J10: LIGHTS, Connector_PinHeader_2.54mm:PinHeader_1x04_P2.54mm_Vertical, symbol Connector:Conn_01x04_Pin
- added J12: Conn_01x02_Pin, Connector_PinHeader_2.54mm:PinHeader_1x02_P2.54mm_Vertical, symbol Connector:Conn_01x02_Pin
- added J13: ATX-24, Connector_Molex:Molex_Mini-Fit_Jr_5569-24A2_2x12_P4.20mm_Horizontal, symbol Connector:ATX-24
- added J8: PELTIER_1, Connector_PinHeader_2.54mm:PinHeader_1x02_P2.54mm_Vertical, symbol Connector:Conn_01x02_Pin
- added J9: PELTIER_2, Connector_PinHeader_2.54mm:PinHeader_1x02_P2.54mm_Vertical, symbol Connector:Conn_01x02_Pin
- added Q6, Q7: DMG6402LVT-7, Package_TO_SOT_SMD:SOT-23-6, symbol Transistor_FET:2N7002E
- added R3, R4, R5: 10K, Resistor_SMD:R_0603_1608Metric, symbol Device:R_US
- J1: footprint (none) -> Connector_PinSocket_2.54mm:PinSocket_1x12_P2.54mm_Vertical; Digikey_Part_Number (none) -> S6100-ND; MPN (none) -> PPTC121LFBN-RC
- J2: footprint (none) -> Connector_PinSocket_2.54mm:PinSocket_1x16_P2.54mm_Vertical; Digikey_Part_Number (none) -> S7014-ND; MPN (none) -> PPTC161LFBN-RC
- J3: value Conn_01x04_Pin -> OUT_FAN_1; footprint (none) -> Connector_PinHeader_2.54mm:PinHeader_1x04_P2.54mm_Vertical; Digikey_Part_Number (none) -> 732-5317-ND; MPN (none) -> 61300411121
- J4: value Conn_01x04_Pin -> OUT_FAN_2; footprint (none) -> Connector_PinHeader_2.54mm:PinHeader_1x04_P2.54mm_Vertical; Digikey_Part_Number (none) -> 732-5317-ND; MPN (none) -> 61300411121
- J5: value Conn_01x04_Pin -> IN_FAN_1; footprint (none) -> Connector_PinHeader_2.54mm:PinHeader_1x04_P2.54mm_Vertical; Digikey_Part_Number (none) -> 732-5317-ND; MPN (none) -> 61300411121
- J6: value Conn_01x04_Pin -> IN_FAN_2; footprint (none) -> Connector_PinHeader_2.54mm:PinHeader_1x04_P2.54mm_Vertical; Digikey_Part_Number (none) -> 732-5317-ND; MPN (none) -> 61300411121
- J7: footprint (none) -> Connector_PinHeader_2.54mm:PinHeader_1x08_P2.54mm_Vertical; Digikey_Part_Number (none) -> 732-5321-ND; MPN (none) -> 61300811121
- Q1: value 2N7002E -> OUT_FAN_1; footprint Package_TO_SOT_SMD:SOT-23 -> Package_TO_SOT_SMD:SOT-23-6; Digikey_Part_Number (none) -> DMG6402LVT-7DICT-ND; MPN (none) -> DMG6402LVT-7
- Q2: value 2N7002E -> OUT_FAN_2; footprint Package_TO_SOT_SMD:SOT-23 -> Package_TO_SOT_SMD:SOT-23-6; Digikey_Part_Number (none) -> DMG6402LVT-7DICT-ND; MPN (none) -> DMG6402LVT-7
- Q3: value 2N7002E -> LIGHTS; footprint Package_TO_SOT_SMD:SOT-23 -> Package_TO_SOT_SMD:SOT-23-6; Digikey_Part_Number (none) -> DMG6402LVT-7DICT-ND; MPN (none) -> DMG6402LVT-7
- Q4: value 2N7002E -> PELTIER_1; footprint Package_TO_SOT_SMD:SOT-23 -> Package_TO_SOT_SMD:SOT-23-6; Digikey_Part_Number (none) -> DMG6402LVT-7DICT-ND; MPN (none) -> DMG6402LVT-7
- Q5: value 2N7002E -> PELTIER_2; footprint Package_TO_SOT_SMD:SOT-23 -> Package_TO_SOT_SMD:SOT-23-6; Digikey_Part_Number (none) -> DMG6402LVT-7DICT-ND; MPN (none) -> DMG6402LVT-7
- R1, R2: footprint (none) -> Resistor_SMD:R_1210_3225Metric; MPN (none) -> CRCW12101K00JNEAIF
Connections:
- net +12V: now also J3.3 (Pin_3), J4.3 (Pin_3), J5.3 (Pin_3), J6.3 (Pin_3), J10.1 (Pin_1), J13.10 (+12V), J13.11 (+12V); no longer J3.1 (Pin_1), J4.1 (Pin_1)
- net +3V3: now also J13.1 (+3.3V), J13.12 (+3.3V), J13.13 (+3.3V), J13.2 (+3.3V); no longer J2.2 (Pin_2), R1.1, R2.1
- net +5V: now also J13.21 (+5V), J13.22 (+5V), J13.23 (+5V), J13.4 (+5V), J13.6 (+5V), J8.1 (Pin_1), J9.1 (Pin_1)
- net GND: now also J5.4 (Pin_4), J6.4 (Pin_4), Q1.4 (S), Q2.4 (S), Q3.4 (S), Q4.4 (S), Q5.4 (S), J12.2 (Pin_2), J13.15 (GND), J13.17 (GND), J13.18 (GND), J13.19 (GND), J13.24 (GND), J13.3 (GND), J13.5 (GND), J13.7 (GND), Q6.4 (S), Q7.4 (S), R3.2, R4.2, R5.2; no longer Q1.2 (S), Q2.2 (S), Q3.2 (S), Q4.2 (S), Q5.2 (S)
- net PWM_FAN_IN_1: now also J5.1 (Pin_1); no longer J5.3 (Pin_3)
- net PWM_FAN_IN_2: now also J6.1 (Pin_1); no longer J6.3 (Pin_3)
- net PWM_L: now also Q3.3 (G), R5.1; no longer Q3.1 (G)
- net TACH_1: now also J5.2 (Pin_2); no longer J5.4 (Pin_4)
- net TACH_2: now also J6.2 (Pin_2); no longer J6.4 (Pin_4)
- net TOGGLE_COOL_1: now also Q1.3 (G), Q4.3 (G), R3.1; no longer Q1.1 (G), Q4.1 (G)
- net TOGGLE_COOL_2: now also Q2.3 (G), Q5.3 (G), R4.1; no longer Q2.1 (G), Q5.1 (G)
- net at J4.2 (Pin_2): no longer Q2.3 (D)
- net at J4.4 (Pin_4): now also Q2.1 (D), Q2.2 (D), Q2.5 (D), Q2.6 (D)
- net at J3.2 (Pin_2): no longer Q1.3 (D)
- net at J3.4 (Pin_4): now also Q1.1 (D), Q1.2 (D), Q1.5 (D), Q1.6 (D)
- net BUTTON_4: no longer names the net of J2.7 (Pin_7)
- new net: J8.2 (Pin_2), Q4.1 (D), Q4.2 (D), Q4.5 (D), Q4.6 (D)
- new net: J10.2 (Pin_2), Q3.1 (D), Q3.2 (D), Q3.5 (D), Q3.6 (D)
- new net: J9.2 (Pin_2), Q5.1 (D), Q5.2 (D), Q5.5 (D), Q5.6 (D)
- new net: J10.3 (Pin_3), Q6.1 (D), Q6.2 (D), Q6.5 (D), Q6.6 (D)
- new net: J10.4 (Pin_4), Q7.1 (D), Q7.2 (D), Q7.5 (D), Q7.6 (D)
- new net PS_ON: J12.1 (Pin_1), J13.16 (PS_ON#)
- new net VCC: J2.2 (Pin_2), R1.1, R2.1
- no-connect marks 20 -> 23
Other:
- note added: "+5VSB (STAND_BY)"
- note added: "12V"
- note added: "4 pin connector options 1. 0022232041 (plastic shroud looks like is on 4 pins) 2. 0022292041 (plastic shroud looks like is on 4 pins) We need plastic shroud on 3 pins 1. 0470533000 - this option should work, BUT, it has a post. That makes it a non-std footprint, which i dont want to deal with - Lets go ahead with this poart for now. Worst case, we can just cut that post. Or make a new FP."
- note added: "ATX connector"
- note added: "Aux Board - for a separate display"
- note added: "Connector_Molex:Molex_Mini-Fit_Jr_5569-24A2_2x12_P4.20mm_Horizontal"
- note added: "Currently we only need 2 pin. But, adding a 4 pin to potentially support a RGB control (R+G+B+GND)"
- note added: "FANS"
- note added: "GND"
- note added: "INSIDE FANS 1. Always powered ON, but speed controlled through PWM signal"
- note added: "LIGHTS"
- note added: "LINK: Check pinout here"
- note added: "LINK:Or buy this"
- note added: "MCU connections"
- note added: "Mosfets: https://www.digikey.com/en/products/detail/diodes-incorporated/DMG6402LDM-7/2179845 https://www.digikey.com/en/products/detail/vishay-siliconix/IRLZ14PBF/811728"
- note added: "Note: The ATX specification requires that the power-good signal ("PWR_OK") go high no sooner than 100 ms after the power rails have stabilized,"
- note added: "OUTSIDE FANS 1. ON when Peltier is powered ON 2. OFF when Peltier is powered OFF"
- note added: "PELTIER"
- note added: "PS-ON is a signal from motherboard to PS to turn ON. Needs to be GNDd to turn on PS."
- note added: "PWM_CONTROL"
- note added: "PWR_OK"
- note added: "Pin cannot be pulled high during boot ToDo: Add source for this comment"
- note added: "Pin mapping can be verfied in software: https://github.com/nitin710/openplant_incubator_fw"
- note added: "Provision for connecting an extention board to hook up https://www.adafruit.com/product/4650"
- note added: "See image for the truth source"
- note added: "TACH"
- note added: "ToDo: Explicitely mark pins as "free to use". Helps future designers to allocate Pins when the design expands."
- note added: "ToDo: verify the polarity of the connector. The pin nets change depending on the perspective (Looking from back or front)"
- note removed: "LIGHT"
- note removed: "LIGHT_B"
- note removed: "LIGHT_G"
- note removed: "LIGHT_R"
- note removed: "NC"
- note removed: "P1"
- note removed: "P2"
- note removed: "Pin cannot be pulled high during boot"
- note removed: "SET_LIGHT_DOWN"
- note removed: "ToDO: 1. Add 24 pin ATX connector 2. Add provision for beakout board for display and input controls - Needs 3v3 from ATX going to the display 3. find switches"
- company: (none) -> Openplant
- title: (none) -> Openplant Incubator mian board
- moved on the sheet: J1, J2, J3, J7, Q1, R1

Commit message: changes
Parts:
- removed J7: Conn_01x08, Connector_PinHeader_2.54mm:PinHeader_1x08_P2.54mm_Vertical, symbol Connector_Generic:Conn_01x08
- added J11: Conn_02x10_Odd_Even, Connector_PinHeader_2.54mm:PinHeader_2x10_P2.54mm_Vertical, symbol Connector_Generic:Conn_02x10_Odd_Even
- added R10, R11, R6, R7, R8, R9: 0R, Resistor_SMD:R_0603_1608Metric, symbol Device:R_US
Connections:
- net +3V3: now also J11.1 (Pin_1)
- net +5V: now also J11.17 (Pin_17)
- net BUTTON_1: now also J11.5 (Pin_5)
- net BUTTON_2: now also J11.7 (Pin_7)
- net BUTTON_3: now also J11.9 (Pin_9)
- net GND: now also J11.19 (Pin_19), J11.3 (Pin_3)
- net PWM_FAN_IN_1: now also R10.1, R7.1; no longer J2.12 (Pin_12)
- net PWM_FAN_IN_2: now also R11.1, R6.1; no longer J2.13 (Pin_13)
- net PWM_L: now also R8.1, R9.1; no longer J2.11 (Pin_11)
- net SCL: now also J11.15 (Pin_15)
- net SDA: now also J11.13 (Pin_13)
- net AO: now reaches J2.5 (Pin_5)
- net AO: now also J11.2 (Pin_2)
- net A1: now reaches J2.6 (Pin_6)
- net A1: now also J11.4 (Pin_4)
- net at J2.7 (Pin_7): now also R9.2
- net at J2.8 (Pin_8): now also R10.2
- net at J2.9 (Pin_9): now also R11.2
- net IO13: now reaches J1.4 (Pin_4)
- net IO13: now also J11.6 (Pin_6)
- net IO12: now reaches J1.5 (Pin_5)
- net IO12: now also J11.8 (Pin_8)
- new net MISO: J11.14 (Pin_14), J2.13 (Pin_13), R6.2
- new net MOSI: J11.12 (Pin_12), J2.12 (Pin_12), R7.2
- new net SCK: J11.10 (Pin_10), J2.11 (Pin_11), R8.2
- no-connect marks 23 -> 19
Other:
- note added: "BUTTON_A"
- note added: "BUTTON_B"
- note added: "BUTTON_C"
- note added: "OLED wing https://www.adafruit.com/product/4650"
- note removed: "Pin cannot be pulled high during boot ToDo: Add source for this comment"
- note removed: "Provision for connecting an extention board to hook up https://www.adafruit.com/product/4650"
- note removed: "SET_LIGHT_UP"
- note removed: "SET_TEMP_DOWN"
- note removed: "SET_TEMP_UP"
- moved on the sheet: J1, J2, R1, R2, R5

Commit message: adding MFG files
Parts:
- R3, R4, R5: Digikey Part Number RMCF0603JT10K0CT-ND -> (none); Digikey_Part_Number (none) -> RMCF0603JT10K0CT-ND
Changed lines of the file:
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@@
 			)
 		)
-		(property "Digikey Part Number" "RMCF0603JT10K0CT-ND"
+		(property "Digikey_Part_Number" "RMCF0603JT10K0CT-ND"
 			(at 207.01 54.61 0)
 			(effects
@@
 			)
 		)
-		(property "Digikey Part Number" "RMCF0603JT10K0CT-ND"
+		(property "Digikey_Part_Number" "RMCF0603JT10K0CT-ND"
 			(at 173.99 129.54 0)
 			(effects
@@
 			)
 		)
-		(property "Digikey Part Number" "RMCF0603JT10K0CT-ND"
+		(property "Digikey_Part_Number" "RMCF0603JT10K0CT-ND"
 			(at 175.26 55.88 0)
 			(effects
